File: Kicad/Arduino.sch (KiCad schematic (older format))
At the start: 1 part

Commit message: update
Connections:
- net at ARD1.26 (AREF): now also ARD1.28 (3V3)
- net Therm_AIN: now reaches ARD1.8 (AnalogIn3)
- net Measure_pH_or_Temp: no longer names the net of ARD1.18 (Digital7)
Other:
- note added: "Pumps not used during sensor readings."
- note added: "Using Arduino's ADC for Thermistor readings. AFEF will use 3.3V."
- note added: "Vin comes from power source. NOT USB"
Changed lines of the file:
@@
 Sheet 2 8
 Title ""
-Date "4 dec 2014"
+Date "8 dec 2014"
 Rev ""
 Comp ""
@@
 Wire Wire Line
 	3550 3050 2450 3050
-Text HLabel 6800 3200 2    60   Output ~ 0
-Measure_pH_or_Temp
 Wire Wire Line
-	5750 3200 6800 3200
+	3550 2150 3050 2150
+Wire Wire Line
+	3050 2150 3050 750
+Wire Wire Line
+	3050 750  5900 750
+Wire Wire Line
+	5900 750  5900 1600
+Wire Wire Line
+	5900 1600 5750 1600
+Text Notes 6150 1150 0    60   ~ 0
+Using Arduino's ADC for Thermistor readings.  AFEF will use 3.3V.
+Text Notes 1300 3350 0    60   ~ 0
+Vin comes from power source.  NOT USB
+Text HLabel 2900 4150 0    60   Input ~ 0
+Therm_AIN
+Wire Wire Line
+	3550 4150 2900 4150
+Text Notes 7450 3650 0    60   ~ 0
+Pumps not used during sensor readings.
 $EndSCHEMATC

Commit message: first pass at layout
Connections:
- net Therm_AIN is gone; now on net ALERT: ARD1.8 (AnalogIn3)
- net ALERT: no longer ARD1.17 (Digital6)
- net Pump1: now also ARD1.18 (Digital7); no longer ARD1.14 (Digital3)
- net Pump2: now also ARD1.19 (Digital8); no longer ARD1.15 (Digital4)
- net Pump3: now also ARD1.20 (PWM0); no longer ARD1.16 (Digital5)
- net at ARD1.26 (AREF): no longer ARD1.28 (3V3)
- net GND_ARD renamed GND
- net V+_ARD: no longer names the net of ARD1.1 (5V)
Other:
- note added: "Vin comes from power source (i.e: Not USB)"
- note removed: "Using Arduino's ADC for Thermistor readings. AFEF will use 3.3V."
- note removed: "Vin comes from power source. NOT USB"
Changed lines of the file:
@@
 Sheet 2 8
 Title ""
-Date "8 dec 2014"
+Date "17 dec 2014"
 Rev ""
 Comp ""
@@
 Comment4 ""
 $EndDescr
-Text HLabel 2500 2450 0    60   Output ~ 0
-V+_ARD
-Wire Wire Line
-	3550 2450 2500 2450
 $Comp
 L ARDUINOPINS ARD1
@@
 	1    0    0    -1
 $EndComp
-Text HLabel 2500 2650 0    60   Input ~ 0
-GND_ARD
 Wire Wire Line
 	2500 2650 3550 2650
 Wire Wire Line
-	6800 3800 5750 3800
+	6800 3000 5750 3000
 Wire Wire Line
-	3550 2850 3200 2850
-Wire Wire Line
-	3200 2850 3200 2650
-Connection ~ 3200 2650
+	2500 2850 3550 2850
 Text HLabel 2900 4350 0    60   BiDi ~ 0
 SDA
@@
 Wire Wire Line
 	2900 4550 3550 4550
-Text HLabel 6800 3800 2    59   Output ~ 0
+Text HLabel 6800 3000 2    59   Output ~ 0
 Pump2
-Text HLabel 6800 4000 2    59   Output ~ 0
+Text HLabel 6800 3200 2    59   Output ~ 0
 Pump1
 Wire Wire Line
-	6800 4000 5750 4000
-Text HLabel 6800 3600 2    59   Output ~ 0
+	6800 3200 5750 3200
+Text HLabel 6800 2800 2    59   Output ~ 0
 Pump3
 Wire Wire Line
-	5750 3600 6800 3600
-Text HLabel 6800 3400 2    59   Input ~ 0
+	5750 2800 6800 2800
+Text HLabel 2850 4150 0    59   Input ~ 0
 ALERT
 Wire Wire Line
-	6800 3400 5750 3400
-Text HLabel 2450 3050 0    60   Output ~ 0
+	3550 3050 2450 3050
+Text Notes 1300 3350 0    60   ~ 0
+Vin comes from power source (i.e: Not USB)
+Text Notes 7450 2850 0    60   ~ 0
+Pumps not used during sensor readings.
+Text GLabel 2500 2650 0    60   Output ~ 0
+GND
+Text GLabel 2450 3050 0    60   Output ~ 0
 Vin
+Text GLabel 2500 2850 0    60   Output ~ 0
+GND
 Wire Wire Line
-	3550 3050 2450 3050
-Wire Wire Line
-	3550 2150 3050 2150
-Wire Wire Line
-	3050 2150 3050 750
-Wire Wire Line
-	3050 750  5900 750
-Wire Wire Line
-	5900 750  5900 1600
-Wire Wire Line
-	5900 1600 5750 1600
-Text Notes 6150 1150 0    60   ~ 0
-Using Arduino's ADC for Thermistor readings.  AFEF will use 3.3V.
-Text Notes 1300 3350 0    60   ~ 0
-Vin comes from power source.  NOT USB
-Text HLabel 2900 4150 0    60   Input ~ 0
-Therm_AIN
-Wire Wire Line
-	3550 4150 2900 4150
-Text Notes 7450 3650 0    60   ~ 0
-Pumps not used during sensor readings.
+	3550 4150 2850 4150
 $EndSCHEMATC

Commit message: 2nd iteration on layout
Connections:
- net ALERT: no longer names the net of ARD1.8 (AnalogIn3)
Changed lines of the file:
@@
 Sheet 2 8
 Title ""
-Date "17 dec 2014"
+Date "18 dec 2014"
 Rev ""
 Comp ""
@@
 Wire Wire Line
 	5750 2800 6800 2800
-Text HLabel 2850 4150 0    59   Input ~ 0
-ALERT
 Wire Wire Line
 	3550 3050 2450 3050
@@
 Text GLabel 2500 2850 0    60   Output ~ 0
 GND
-Wire Wire Line
-	3550 4150 2850 4150
 $EndSCHEMATC
