File: Kicad/Arduino.sch (KiCad schematic (older format))
At the start: 1 part

Commit message: iPhone app and changes to hw design (not sure I like)
Connections:
- net Pump3 is gone; now on net MUX_out_pin: ARD1.20 (PWM0)
- net FET_pin: now also ARD1.16 (Digital5); no longer ARD1.6 (AnalogIn1)
- net MUX_out_pin: no longer ARD1.8 (AnalogIn3)
- net Vclean: now reaches ARD1.1 (5V)
- net Pump1_SW: now reaches ARD1.17 (Digital6)
- net MUX_enable_pin: no longer names the net of ARD1.7 (AnalogIn2)
- net Pump1 renamed Pump2_SW
- net Pump2 renamed Pump3_SW
- net Vin renamed 12V
Other:
- note removed: "Pumps not used during sensor readings."
- note removed: "Vin comes from power source (i.e: Not USB)"
Changed lines of the file:
@@
 $Descr A4 11693 8268
 encoding utf-8
-Sheet 2 11
+Sheet 2 9
 Title ""
-Date "9 feb 2015"
+Date "17 mar 2015"
 Rev ""
 Comp ""
@@
 	2500 2650 3550 2650
 Wire Wire Line
-	6800 3000 5750 3000
-Wire Wire Line
 	2500 2850 3550 2850
 Text HLabel 2900 4350 0    60   BiDi ~ 0
@@
 Wire Wire Line
 	2900 4550 3550 4550
-Text HLabel 6800 3000 2    59   Output ~ 0
-Pump2
-Text HLabel 6800 3200 2    59   Output ~ 0
-Pump1
-Wire Wire Line
-	6800 3200 5750 3200
-Text HLabel 6800 2800 2    59   Output ~ 0
-Pump3
-Wire Wire Line
-	5750 2800 6800 2800
-Wire Wire Line
-	3550 3050 2450 3050
-Text Notes 1300 3350 0    60   ~ 0
-Vin comes from power source (i.e: Not USB)
-Text Notes 7450 2850 0    60   ~ 0
-Pumps not used during sensor readings.
 Text GLabel 2500 2650 0    60   Output ~ 0
 GND
-Text GLabel 2450 3050 0    60   Output ~ 0
-Vin
 Text GLabel 2500 2850 0    60   Output ~ 0
 GND
-Text HLabel 2850 4150 0    60   Output ~ 0
+Text HLabel 7100 2800 2    60   Output ~ 0
 MUX_out_pin
-Text HLabel 2850 3750 0    60   Output ~ 0
+Text HLabel 7100 3600 2    60   Output ~ 0
 FET_pin
+Text GLabel 2500 2450 0    60   Output ~ 0
+Vclean
 Wire Wire Line
-	2850 4150 3550 4150
+	3550 2450 2500 2450
 Wire Wire Line
-	3550 3950 2850 3950
-Text HLabel 2850 3950 0    60   Output ~ 0
-MUX_enable_pin
+	1600 3050 3550 3050
+Text HLabel 1600 3050 0    60   Input ~ 0
+12V
 Wire Wire Line
-	2850 3750 3550 3750
+	5750 3600 7100 3600
+Text HLabel 7100 3400 2    60   Output ~ 0
+Pump1_SW
+Wire Wire Line
+	7100 3400 5750 3400
+Text HLabel 7100 3200 2    60   Output ~ 0
+Pump2_SW
+Text HLabel 7100 3000 2    60   Output ~ 0
+Pump3_SW
+Wire Wire Line
+	5750 3000 7100 3000
+Wire Wire Line
+	5750 3200 7100 3200
+Wire Wire Line
+	5750 2800 7100 2800
 $EndSCHEMATC
