File: Kicad/Arduino.sch (KiCad schematic (older format))
At the start: 1 part

Commit message: added ECTest Arduino Sketch also updates (not all) to the Schematic
Connections:
- net EC_Meas_Switch: now reaches ARD1.17 (Digital6)
Changed lines of the file:
@@
 $Descr A4 11693 8268
 encoding utf-8
-Sheet 2 8
+Sheet 2 11
 Title ""
-Date "21 jan 2015"
+Date "29 jan 2015"
 Rev ""
 Comp ""
@@
 Text GLabel 2500 2850 0    60   Output ~ 0
 GND
+Text HLabel 6800 3400 2    60   Output ~ 0
+EC_Meas_Switch
+Wire Wire Line
+	5750 3400 6800 3400
 $EndSCHEMATC

Commit message: layout for Alpha 2
Connections:
- net FET_pin: now reaches ARD1.6 (AnalogIn1)
- net MUX_enable_pin: now reaches ARD1.7 (AnalogIn2)
- net MUX_out_pin: now reaches ARD1.8 (AnalogIn3)
- net EC_Meas_Switch: no longer names the net of ARD1.17 (Digital6)
Changed lines of the file:
@@
 Sheet 2 11
 Title ""
-Date "29 jan 2015"
+Date "8 feb 2015"
 Rev ""
 Comp ""
@@
 Text GLabel 2500 2850 0    60   Output ~ 0
 GND
-Text HLabel 6800 3400 2    60   Output ~ 0
-EC_Meas_Switch
+Text HLabel 2850 4150 0    60   Output ~ 0
+MUX_out_pin
+Text HLabel 2850 3750 0    60   Output ~ 0
+FET_pin
 Wire Wire Line
-	5750 3400 6800 3400
+	2850 4150 3550 4150
+Wire Wire Line
+	3550 3950 2850 3950
+Text HLabel 2850 3950 0    60   Output ~ 0
+MUX_enable_pin
+Wire Wire Line
+	2850 3750 3550 3750
 $EndSCHEMATC

Commit message: Beta 2 sent to OSHPark
Parts:
- added D8: LED, ~, symbol LED
- added P2, P5: CONN_2, symbol CONN_2
- added R2: 1K, ~, symbol R
Connections:
- net GND: now also P2.2 (PM), R2.1
- net Vclean: now reaches ARD1.1 (5V)
- net MUX_enable_pin: no longer names the net of ARD1.7 (AnalogIn2)
- net Pump1 renamed pump1_pin
- net Pump2 renamed pump2_pin
- net Pump3 renamed pump3_pin
- net Vin renamed 12V
- net 12V: now also D8.1 (A), P5.1 (P1)
- new net: D8.2 (K), R2.2
- new net 12Va: P2.1 (P1), P5.2 (PM)
Other:
- note removed: "Pumps not used during sensor readings."
- note removed: "Vin comes from power source (i.e: Not USB)"
Changed lines of the file:
@@
 $Descr A4 11693 8268
 encoding utf-8
-Sheet 2 11
+Sheet 2 10
 Title ""
-Date "9 feb 2015"
+Date "26 mar 2015"
 Rev ""
 Comp ""
@@
 $EndComp
 Wire Wire Line
-	2500 2650 3550 2650
-Wire Wire Line
 	6800 3000 5750 3000
-Wire Wire Line
-	2500 2850 3550 2850
 Text HLabel 2900 4350 0    60   BiDi ~ 0
 SDA
@@
 	2900 4550 3550 4550
 Text HLabel 6800 3000 2    59   Output ~ 0
-Pump2
+pump2_pin
 Text HLabel 6800 3200 2    59   Output ~ 0
-Pump1
+pump1_pin
 Wire Wire Line
 	6800 3200 5750 3200
 Text HLabel 6800 2800 2    59   Output ~ 0
-Pump3
+pump3_pin
 Wire Wire Line
 	5750 2800 6800 2800
-Wire Wire Line
-	3550 3050 2450 3050
-Text Notes 1300 3350 0    60   ~ 0
-Vin comes from power source (i.e: Not USB)
-Text Notes 7450 2850 0    60   ~ 0
-Pumps not used during sensor readings.
-Text GLabel 2500 2650 0    60   Output ~ 0
-GND
-Text GLabel 2450 3050 0    60   Output ~ 0
-Vin
-Text GLabel 2500 2850 0    60   Output ~ 0
-GND
 Text HLabel 2850 4150 0    60   Output ~ 0
 MUX_out_pin
@@
 	2850 4150 3550 4150
 Wire Wire Line
-	3550 3950 2850 3950
-Text HLabel 2850 3950 0    60   Output ~ 0
-MUX_enable_pin
+	2850 3750 3550 3750
 Wire Wire Line
-	2850 3750 3550 3750
+	2500 2650 3550 2650
+Wire Wire Line
+	1500 2850 3550 2850
+Text GLabel 2500 2650 0    60   Output ~ 0
+GND
+Text GLabel 2500 2450 0    60   Output ~ 0
+Vclean
+Wire Wire Line
+	3550 2450 2500 2450
+Text HLabel 3050 3250 0    60   Output ~ 0
+12V
+$Comp
+L CONN_2 P5
+U 1 1 5512F560
+P 2150 3400
+F 0 "P5" V 2100 3400 40  0000 C CNN
+F 1 "CONN_2" V 2200 3400 40  0000 C CNN
+F 2 "" H 2150 3400 60  0000 C CNN
+F 3 "" H 2150 3400 60  0000 C CNN
+	1    2150 3400
+	0    1    1    0
+$EndComp
+$Comp
+L CONN_2 P2
+U 1 1 5512F566
+P 1150 2950
+F 0 "P2" V 1100 2950 40  0000 C CNN
+F 1 "CONN_2" V 1200 2950 40  0000 C CNN
+F 2 "" H 1150 2950 60  0000 C CNN
+F 3 "" H 1150 2950 60  0000 C CNN
+	1    1150 2950
+	-1   0    0    1
+$EndComp
+Wire Wire Line
+	3550 3050 2250 3050
+Wire Wire Line
+	2050 3050 1500 3050
+Wire Wire Line
+	3250 2650 3250 2850
+Connection ~ 3250 2850
+Connection ~ 3250 2650
+Wire Wire Line
+	3050 3250 3050 3050
+Connection ~ 3050 3050
+Text Label 1600 3050 0    60   ~ 0
+12Va
+$Comp
+L LED D8
+U 1 1 551317CB
+P 1350 4200
+F 0 "D8" H 1350 4300 50  0000 C CNN
+F 1 "LED" H 1350 4100 50  0000 C CNN
+F 2 "~" H 1350 4200 60  0000 C CNN
+F 3 "~" H 1350 4200 60  0000 C CNN
+	1    1350 4200
+	0    1    1    0
+$EndComp
+$Comp
+L R R2
+U 1 1 551317D1
+P 1350 4800
+F 0 "R2" V 1430 4800 40  0000 C CNN
+F 1 "1K" V 1357 4801 40  0000 C CNN
+F 2 "~" V 1280 4800 30  0000 C CNN
+F 3 "~" H 1350 4800 30  0000 C CNN
+	1    1350 4800
+	-1   0    0    1
+$EndComp
+Wire Wire Line
+	1350 4400 1350 4550
+Wire Wire Line
+	1350 3650 1350 4000
+Wire Wire Line
+	1350 5050 1350 5350
+Wire Wire Line
+	2650 3050 2600 3650
+Wire Wire Line
+	2600 3650 1350 3650
+Connection ~ 2650 3050
+Text GLabel 1100 5350 0    60   Output ~ 0
+GND
+Wire Wire Line
+	1350 5350 1100 5350
 $EndSCHEMATC

Commit message: minor changes - all works
Parts:
- removed P2, P5: CONN_2, symbol CONN_2
Changed lines of the file:
@@
 Sheet 2 10
 Title ""
-Date "26 mar 2015"
+Date "13 apr 2015"
 Rev ""
 Comp ""
@@
 Wire Wire Line
 	2500 2650 3550 2650
-Wire Wire Line
-	1500 2850 3550 2850
 Text GLabel 2500 2650 0    60   Output ~ 0
 GND
@@
 Wire Wire Line
 	3550 2450 2500 2450
-Text HLabel 3050 3250 0    60   Output ~ 0
+Text HLabel 950  3050 0    60   Output ~ 0
 12V
-$Comp
-L CONN_2 P5
-U 1 1 5512F560
-P 2150 3400
-F 0 "P5" V 2100 3400 40  0000 C CNN
-F 1 "CONN_2" V 2200 3400 40  0000 C CNN
-F 2 "" H 2150 3400 60  0000 C CNN
-F 3 "" H 2150 3400 60  0000 C CNN
-	1    2150 3400
-	0    1    1    0
-$EndComp
-$Comp
-L CONN_2 P2
-U 1 1 5512F566
-P 1150 2950
-F 0 "P2" V 1100 2950 40  0000 C CNN
-F 1 "CONN_2" V 1200 2950 40  0000 C CNN
-F 2 "" H 1150 2950 60  0000 C CNN
-F 3 "" H 1150 2950 60  0000 C CNN
-	1    1150 2950
-	-1   0    0    1
-$EndComp
 Wire Wire Line
-	3550 3050 2250 3050
-Wire Wire Line
-	2050 3050 1500 3050
+	950  3050 3550 3050
 Wire Wire Line
 	3250 2650 3250 2850
-Connection ~ 3250 2850
 Connection ~ 3250 2650
-Wire Wire Line
-	3050 3250 3050 3050
-Connection ~ 3050 3050
-Text Label 1600 3050 0    60   ~ 0
-12Va
 $Comp
 L LED D8
@@
 	1350 4400 1350 4550
 Wire Wire Line
-	1350 3650 1350 4000
+	1350 3050 1350 4000
 Wire Wire Line
 	1350 5050 1350 5350
-Wire Wire Line
-	2650 3050 2600 3650
-Wire Wire Line
-	2600 3650 1350 3650
-Connection ~ 2650 3050
 Text GLabel 1100 5350 0    60   Output ~ 0
 GND
 Wire Wire Line
 	1350 5350 1100 5350
+Connection ~ 1350 3050
+Wire Wire Line
+	3250 2850 3550 2850
 $EndSCHEMATC
