File: Kicad/DigitalAccess.sch (KiCad schematic (older format))
At the start: 4 parts

Commit message: update
Connections:
- net EC_AIN: now also U?.6 (AIN2)
- net VGND: now also U?.5 (AIN1), U?.7 (AIN3)
- net pH_AIN: now also U?.4 (AIN0)
Changed lines of the file:
@@
 Sheet 3 8
 Title ""
-Date "4 dec 2014"
+Date "8 dec 2014"
 Rev ""
 Comp ""
@@
 Wire Wire Line
 	3850 4050 3550 4050
-Text HLabel 7100 2900 2    60   Input ~ 0
+Text HLabel 6000 3150 2    60   Input ~ 0
 pH_AIN
-Text HLabel 7100 3150 2    60   Input ~ 0
+Text HLabel 6000 3450 2    60   Input ~ 0
 EC_AIN
-Text HLabel 7150 3450 2    60   Input ~ 0
-Therm_AIN
-Text HLabel 7200 3750 2    60   Input ~ 0
+Text HLabel 6000 3300 2    60   Input ~ 0
 VGND
 Text Notes 8200 2050 2    60   ~ 0
 TBD: MUX to switch between pH and  Thermistor AIN
-Text HLabel 7050 4200 2    60   Input ~ 0
-Measure_pH_or_Temp
+Wire Wire Line
+	5250 3150 6000 3150
+Wire Wire Line
+	5250 3300 6000 3300
+Wire Wire Line
+	5250 3450 6000 3450
+Text HLabel 6000 3600 2    60   Input ~ 0
+VGND
+Wire Wire Line
+	5250 3600 6000 3600
 $EndSCHEMATC

Commit message: first pass at layout
Parts:
- R7: renamed from 10K; value 3K -> 10K
- gave numbers to parts that had none: 1
Connections:
- net AGND is gone; now on net GND: U4.1 (ADDR), U4.3 (AGND)
- net EC_AIN: now also U4.5 (AIN1); no longer U4.6 (AIN2)
- net VGND: no longer U4.5 (AIN1)
- net GND: now reaches C1.2
- net GND: no longer U4.8 (V+)
- net V+_WallWart renamed Vclean
- net Vclean: now also U4.8 (V+)
- new net Therm_AIN: U4.6 (AIN2)
Other:
- note removed: "TBD: MUX to switch between pH and Thermistor AIN"
- moved on the sheet: C1
Changed lines of the file:
@@
 Sheet 3 8
 Title ""
-Date "8 dec 2014"
+Date "17 dec 2014"
 Rev ""
 Comp ""
@@
 $EndComp
 $Comp
-L R 10K
+L R R7
 U 1 1 5463DA60
 P 3550 2400
-F 0 "10K" V 3630 2400 40  0000 C CNN
-F 1 "3K" V 3557 2401 40  0000 C CNN
+F 0 "R7" V 3630 2400 40  0000 C CNN
+F 1 "10K" V 3557 2401 40  0000 C CNN
 F 2 "~" V 3480 2400 30  0000 C CNN
 F 3 "~" H 3550 2400 30  0000 C CNN
@@
 	1    0    0    -1
 $EndComp
-Text HLabel 2400 2100 0    60   Input ~ 0
-V+_WallWart
 $Comp
 L C C1
 U 1 1 546637F5
-P 5250 2450
-F 0 "C1" H 5250 2550 40  0000 L CNN
-F 1 ".1u" H 5256 2365 40  0000 L CNN
-F 2 "~" H 5288 2300 30  0000 C CNN
-F 3 "~" H 5250 2450 60  0000 C CNN
-	1    5250 2450
+P 5700 2500
+F 0 "C1" H 5700 2600 40  0000 L CNN
+F 1 ".1u" H 5706 2415 40  0000 L CNN
+F 2 "~" H 5738 2350 30  0000 C CNN
+F 3 "~" H 5700 2500 60  0000 C CNN
+	1    5700 2500
 	1    0    0    -1
 $EndComp
@@
 	3850 3650 3850 4050
 Wire Wire Line
-	2400 2100 5250 2100
+	2400 2100 5700 2100
 Wire Wire Line
 	3550 2100 3550 2150
@@
 	3850 3150 2400 3150
 $Comp
-L ADS1015 U?
+L ADS1015 U4
 U 1 1 54804BC7
 P 4550 3300
-F 0 "U?" H 4750 3850 60  0000 L CNN
+F 0 "U4" H 4750 3850 60  0000 L CNN
 F 1 "ADS1015" H 4700 2750 60  0000 L CNN
 F 2 "" H 4550 3300 60  0000 C CNN
@@
 Connection ~ 3200 3150
 Wire Wire Line
-	5250 2950 5250 2650
-Wire Wire Line
-	5250 2100 5250 2250
+	5250 2100 5250 2950
 Connection ~ 3550 2100
-Text HLabel 3550 4050 0    60   Output ~ 0
-AGND
 Wire Wire Line
 	3850 4050 3550 4050
 Text HLabel 6000 3150 2    60   Input ~ 0
 pH_AIN
-Text HLabel 6000 3450 2    60   Input ~ 0
+Text HLabel 6000 3300 2    60   Input ~ 0
 EC_AIN
-Text HLabel 6000 3300 2    60   Input ~ 0
-VGND
-Text Notes 8200 2050 2    60   ~ 0
-TBD: MUX to switch between pH and  Thermistor AIN
 Wire Wire Line
 	5250 3150 6000 3150
@@
 Wire Wire Line
 	5250 3450 6000 3450
-Text HLabel 6000 3600 2    60   Input ~ 0
-VGND
 Wire Wire Line
 	5250 3600 6000 3600
+Wire Wire Line
+	5700 2100 5700 2300
+Connection ~ 5250 2100
+Text GLabel 6000 3600 2    60   Input ~ 0
+VGND
+Text GLabel 3550 4050 0    60   Output ~ 0
+GND
+Text GLabel 5800 2800 2    60   Output ~ 0
+GND
+Wire Wire Line
+	5700 2700 5700 2800
+Wire Wire Line
+	5700 2800 5800 2800
+Text GLabel 2400 2100 0    60   Input ~ 0
+Vclean
+Text HLabel 6000 3450 2    60   Input ~ 0
+Therm_AIN
 $EndSCHEMATC

Commit message: 2nd iteration on layout
Connections:
- net ALERT: no longer names the net of U4.2 (ALERT)
Changed lines of the file:
@@
 Sheet 3 8
 Title ""
-Date "17 dec 2014"
+Date "18 dec 2014"
 Rev ""
 Comp ""
@@
 Connection ~ 3850 3800
 Wire Wire Line
-	3850 3300 2400 3300
-Text HLabel 2400 3300 0    60   Output ~ 0
-ALERT
-Wire Wire Line
 	3200 2650 3200 3150
