File: Kicad/DigitalAccess.sch (KiCad schematic (older format))
At the start: 4 parts, among them U4 ADS1015

Commit message: first pass at new layout
Parts:
- U4: footprint (none) -> ~
Changed lines of the file:
@@
 Sheet 3 11
 Title ""
-Date "31 jan 2015"
+Date "2 feb 2015"
 Rev ""
 Comp ""
@@
 Wire Wire Line
 	3850 3150 2400 3150
-$Comp
-L ADS1015 U4
-U 1 1 54804BC7
-P 4550 3300
-F 0 "U4" H 4750 3850 60  0000 L CNN
-F 1 "ADS1015" H 4700 2750 60  0000 L CNN
-F 2 "" H 4550 3300 60  0000 C CNN
-F 3 "" H 4550 3300 60  0000 C CNN
-	1    4550 3300
-	1    0    0    -1
-$EndComp
 Wire Wire Line
 	3850 3800 3700 3800
@@
 Text HLabel 6000 3450 2    60   Input ~ 0
 Therm_AIN
+$Comp
+L ADS1015 U4
+U 1 1 54CE4504
+P 4550 3300
+F 0 "U4" H 4750 3850 60  0000 L CNN
+F 1 "ADS1015" H 4700 2750 60  0000 L CNN
+F 2 "~" H 4550 3300 60  0000 C CNN
+F 3 "~" H 4550 3300 60  0000 C CNN
+	1    4550 3300
+	1    0    0    -1
+$EndComp
 $EndSCHEMATC
