File: Kicad/DigitalAccess.sch (KiCad schematic (older format))
At the start: 4 parts, among them U4 ADS1015

Commit message: iPhone app and changes to hw design (not sure I like)
Connections:
- net Therm_AIN: no longer names the net of U4.6 (AIN2)
Changed lines of the file:
@@
 $Descr A4 11693 8268
 encoding utf-8
-Sheet 3 11
+Sheet 3 9
 Title ""
-Date "9 feb 2015"
+Date "17 mar 2015"
 Rev ""
 Comp ""
@@
 	5250 3300 6000 3300
 Wire Wire Line
-	5250 3450 6000 3450
-Wire Wire Line
 	5250 3600 6000 3600
 Wire Wire Line
@@
 Text GLabel 2400 2100 0    60   Input ~ 0
 Vclean
-Text HLabel 6000 3450 2    60   Input ~ 0
-Therm_AIN
 $EndSCHEMATC
