File: Kicad/Power.sch (KiCad schematic (older format))
At the start: 11 parts, among them U3 MC78L05

Commit message: update
Connections:
- wire segments 36 -> 35
Changed lines of the file:
@@
 Sheet 7 8
 Title ""
-Date "4 dec 2014"
+Date "8 dec 2014"
 Rev ""
 Comp ""
@@
 	5600 4100 5600 3750
 Wire Wire Line
-	2850 4100 7200 4100
+	2850 4100 10050 4100
 Wire Wire Line
 	7200 4100 7200 3950
@@
 	7700 3900 7700 4150
 Wire Wire Line
-	7700 4650 7700 4900
+	7700 4650 7700 5100
 $Comp
 L MC78L05 U3
@@
 AGND
 Wire Wire Line
-	7500 5100 7700 5100
-Wire Wire Line
-	7700 5100 7700 4900
-Connection ~ 5250 4100
+	7700 5100 7500 5100
+Connection ~ 7200 4100
+Text HLabel 10050 4100 2    60   Output ~ 0
+AGND
 $EndSCHEMATC

Commit message: first pass at layout
Parts:
- removed C?: .1u, ~, symbol C
- removed U?: MCP6244, ~, symbol MCP6244
- added C9: .1u, ~, symbol C
- added U2: MCP6242, ~, symbol MCP6242
- gave numbers to parts that had none: 3
Connections:
- net labels added: GND, VGND_V+, Vclean
- net labels removed: AGND, GND_ARD, V+_WallWart, pin 3
- wire segments 35 -> 30
Other:
- note added: "Provide clean V+ to circuit"
- note removed: "For discussion (see pdf on ground planes)"
- moved on the sheet: C11, C12, C13, C4, D3, R5, R8, R9
