File: Kicad/Pumps.sch (KiCad schematic (older format))
At the start: 9 parts, among them Q1 TIP122, Q2 TIP122

Commit message: first pass at layout
Parts:
- gave numbers to parts that had none: 3
Connections:
- net labels added: VClean
- net labels removed: GND_ARD, V+_ARD
Changed lines of the file:
@@
 $Descr A4 11693 8268
 encoding utf-8
-Sheet 6 8
+Sheet 8 8
 Title ""
-Date "8 dec 2014"
+Date "17 dec 2014"
 Rev ""
 Comp ""
@@
 Text HLabel 2000 2650 0    59   Input ~ 0
 Pump1
-$Comp
-L GND #PWR06
-U 1 1 53DC3138
-P 3900 3250
-F 0 "#PWR06" H 3900 3250 30  0001 C CNN
-F 1 "GND" H 3900 3180 30  0001 C CNN
-F 2 "" H 3900 3250 60  0000 C CNN
-F 3 "" H 3900 3250 60  0000 C CNN
-	1    3900 3250
-	1    0    0    -1
-$EndComp
-Text HLabel 1750 1700 0    60   Input ~ 0
-V+_ARD
-Text HLabel 2000 3150 0    59   Output ~ 0
-GND_ARD
 Text HLabel 6000 1700 2    60   Input ~ 0
 V+_Pump1
@@
 Text HLabel 2000 4150 0    59   Input ~ 0
 Pump2
-$Comp
-L GND #PWR07
-U 1 1 53EA6E1E
-P 3900 4750
-F 0 "#PWR07" H 3900 4750 30  0001 C CNN
-F 1 "GND" H 3900 4680 30  0001 C CNN
-F 2 "" H 3900 4750 60  0000 C CNN
-F 3 "" H 3900 4750 60  0000 C CNN
-	1    3900 4750
-	1    0    0    -1
-$EndComp
 Text HLabel 6000 3850 2    60   Input ~ 0
 SW_Pump2
@@
 Connection ~ 5650 2350
 $Comp
-L TIP120 Q?
+L TIP120 Q3
 U 1 1 54803643
 P 3800 5600
-F 0 "Q?" H 3750 5450 40  0000 R CNN
+F 0 "Q3" H 3750 5450 40  0000 R CNN
 F 1 "TIP122" H 3800 5750 40  0000 R CNN
 F 2 "TO220" H 3680 5705 29  0001 C CNN
@@
 $EndComp
 $Comp
-L R R?
+L R R10
 U 1 1 54803649
 P 3100 5600
-F 0 "R?" V 3180 5600 40  0000 C CNN
+F 0 "R10" V 3180 5600 40  0000 C CNN
 F 1 "2.2K" V 3107 5601 40  0000 C CNN
 F 2 "~" V 3030 5600 30  0000 C CNN
@@
 Text HLabel 2000 5600 0    59   Input ~ 0
 Pump3
-$Comp
-L GND #PWR?
-U 1 1 54803650
-P 3900 6200
-F 0 "#PWR?" H 3900 6200 30  0001 C CNN
-F 1 "GND" H 3900 6130 30  0001 C CNN
-F 2 "" H 3900 6200 60  0000 C CNN
-F 3 "" H 3900 6200 60  0000 C CNN
-	1    3900 6200
-	1    0    0    -1
-$EndComp
 Text HLabel 6000 5300 2    60   Input ~ 0
 SW_Pump3
 $Comp
-L DIODE D?
+L DIODE D2
 U 1 1 54803657
 P 5650 5000
-F 0 "D?" H 5650 5100 40  0000 C CNN
+F 0 "D2" H 5650 5100 40  0000 C CNN
 F 1 "4004" H 5650 4900 40  0000 C CNN
 F 2 "~" H 5650 5000 60  0000 C CNN
@@
 	5650 4800 5650 4250
 Connection ~ 5650 4250
+Text GLabel 2000 3150 0    60   Output ~ 0
+GND
+Text GLabel 1750 1700 0    60   Input ~ 0
+VClean
+Text GLabel 3900 3250 2    60   Input ~ 0
+GND
+Text GLabel 3900 4750 2    60   Input ~ 0
+GND
+Text GLabel 3900 6200 2    60   Input ~ 0
+GND
 $EndSCHEMATC
