File: Kicad/Pumps.sch (KiCad schematic (older format))
At the start: 9 parts, among them Q1 TIP122, Q2 TIP122, Q3 TIP122

Commit message: Beta 2 sent to OSHPark
Connections:
- net labels added: 12V, pump1, pump1_pin, pump2, pump2_pin, pump3, pump3_pin
- net labels removed: Pump1, Pump2, Pump3, SW_Pump1, SW_Pump2, SW_Pump3, V+_Pump1, V+_Pump2, V+_Pump3, VClean
- wire segments 29 -> 27
Other:
- moved on the sheet: D2
Changed lines of the file:
@@
 $Descr A4 11693 8268
 encoding utf-8
-Sheet 8 11
+Sheet 10 10
 Title ""
-Date "9 feb 2015"
+Date "26 mar 2015"
 Rev ""
 Comp ""
@@
 $EndComp
 Text HLabel 2000 2650 0    59   Input ~ 0
-Pump1
-Text HLabel 6000 1700 2    60   Input ~ 0
-V+_Pump1
-Text HLabel 6000 2350 2    60   Input ~ 0
-SW_Pump1
+pump1_pin
+Text HLabel 6000 2350 2    60   Output ~ 0
+pump1
 $Comp
 L TIP120 Q2
@@
 $EndComp
 Text HLabel 2000 4150 0    59   Input ~ 0
-Pump2
-Text HLabel 6000 3850 2    60   Input ~ 0
-SW_Pump2
-Text HLabel 6000 3200 2    60   Input ~ 0
-V+_Pump2
+pump2_pin
+Text HLabel 6000 3850 2    60   Output ~ 0
+pump2
 $Comp
 L DIODE D5
@@
 	3900 2350 3900 2450
 Wire Wire Line
-	1750 1700 6000 1700
-Wire Wire Line
 	3900 2850 3900 3250
 Wire Wire Line
@@
 	3900 4350 3900 4750
 Wire Wire Line
-	5300 1700 5300 4250
-Wire Wire Line
-	5300 3200 6000 3200
-Connection ~ 5300 1700
+	5300 1700 5300 4800
 Wire Wire Line
 	2550 3150 2550 6050
@@
 Wire Wire Line
 	5650 3350 5650 3200
-Connection ~ 5650 3200
 Wire Wire Line
 	5650 3750 5650 3850
 Connection ~ 5650 3850
 Wire Wire Line
-	5650 1850 5650 1700
-Connection ~ 5650 1700
+	5650 1700 5650 1850
 Wire Wire Line
 	5650 2250 5650 2350
@@
 $EndComp
 Text HLabel 2000 5600 0    59   Input ~ 0
-Pump3
-Text HLabel 6000 5300 2    60   Input ~ 0
-SW_Pump3
+pump3_pin
+Text HLabel 6000 5300 2    60   Output ~ 0
+pump3
 $Comp
 L DIODE D2
 U 1 1 54803657
-P 5650 5000
-F 0 "D2" H 5650 5100 40  0000 C CNN
-F 1 "4004" H 5650 4900 40  0000 C CNN
-F 2 "~" H 5650 5000 60  0000 C CNN
-F 3 "~" H 5650 5000 60  0000 C CNN
-	1    5650 5000
+P 5300 5000
+F 0 "D2" H 5300 5100 40  0000 C CNN
+F 1 "4004" H 5300 4900 40  0000 C CNN
+F 2 "~" H 5300 5000 60  0000 C CNN
+F 3 "~" H 5300 5000 60  0000 C CNN
+	1    5300 5000
 	0    -1   -1   0
 $EndComp
@@
 	2550 6050 3900 6050
 Connection ~ 3900 6050
-Wire Wire Line
-	5650 5200 5650 5300
-Connection ~ 5650 5300
-Wire Wire Line
-	5300 4250 6050 4250
-Connection ~ 5300 3200
-Text HLabel 6050 4250 2    60   Input ~ 0
-V+_Pump3
-Wire Wire Line
-	5650 4800 5650 4250
-Connection ~ 5650 4250
 Text GLabel 2000 3150 0    60   Output ~ 0
 GND
-Text GLabel 1750 1700 0    60   Input ~ 0
-VClean
 Text GLabel 3900 3250 2    60   Input ~ 0
 GND
@@
 Text GLabel 3900 6200 2    60   Input ~ 0
 GND
+Text HLabel 1700 1700 0    60   Input ~ 0
+12V
+Wire Wire Line
+	5650 3200 5300 3200
+Connection ~ 5300 3200
+Wire Wire Line
+	5300 5200 5300 5300
+Connection ~ 5300 5300
+Wire Wire Line
+	1700 1700 5650 1700
+Connection ~ 5300 1700
 $EndSCHEMATC
