File: Kicad/pH.sch (KiCad schematic (older format))
At the start: 2 parts, among them U1 MCP6241

Commit message: first pass at layout
Parts:
- removed C9: .1, ~, symbol C
- removed U1: MCP6241, ~, symbol MCP6241
- added U2: MCP6242, ~, symbol MCP6242
Connections:
- net labels added: VGND
- net labels removed: AGND, V+_WallWart, pin 4
- wire segments 14 -> 8
Other:
- note added: "Probe"
Changed lines of the file:
@@
 Sheet 4 8
 Title ""
-Date "8 dec 2014"
+Date "17 dec 2014"
 Rev ""
 Comp ""
@@
 Text HLabel 1750 3200 0    60   Output ~ 0
 pH_AIN
-Text HLabel 3600 2300 0    60   Input ~ 0
-V+_WallWart
 Wire Wire Line
-	4150 3100 5700 3100
+	4150 3100 5900 3100
 Wire Wire Line
 	2950 4100 4750 4100
@@
 	4750 3300 4150 3300
 Wire Wire Line
-	3900 2300 3900 2900
-Wire Wire Line
-	3550 2500 3550 2450
-Wire Wire Line
-	3550 2450 3900 2450
-Connection ~ 3900 2450
-Wire Wire Line
 	1750 3200 3450 3200
 Wire Wire Line
 	2950 4100 2950 3200
 Connection ~ 2950 3200
-Text Label 4750 3800 0    60   ~ 0
-pin 4
-Text HLabel 4050 3750 2    60   Output ~ 0
-AGND
-Text HLabel 3400 2950 0    60   Output ~ 0
-AGND
+Text HLabel 5900 3100 2    60   Input ~ 0
+pH_ProbeIN
+Text Notes 6050 3300 2    60   ~ 0
+Probe
+Wire Notes Line
+	5800 3100 6100 3100
+Wire Notes Line
+	6100 3750 5750 3750
+Wire Notes Line
+	5750 3750 5750 3100
+Wire Notes Line
+	5750 3100 5900 3100
+Wire Notes Line
+	6100 3100 6100 3750
+Wire Notes Line
+	5650 3650 6250 3250
+Wire Notes Line
+	6250 3250 6250 3350
+Wire Notes Line
+	6250 3250 6150 3250
 Wire Wire Line
-	3600 2300 3900 2300
+	5900 3750 5900 4150
+Wire Wire Line
+	5900 4150 6050 4150
+Text GLabel 6050 4150 2    60   Input ~ 0
+VGND
 $Comp
-L C C9
-U 1 1 54453E50
-P 3550 2700
-F 0 "C9" H 3550 2800 40  0000 L CNN
-F 1 ".1" H 3556 2615 40  0000 L CNN
-F 2 "~" H 3588 2550 30  0000 C CNN
-F 3 "~" H 3550 2700 60  0000 C CNN
-	1    3550 2700
-	1    0    0    -1
-$EndComp
-Wire Wire Line
-	3550 2950 3400 2950
-Wire Wire Line
-	3550 2950 3550 2900
-Wire Wire Line
-	3900 3750 4050 3750
-Wire Wire Line
-	3900 3500 3900 3750
-$Comp
-L MCP6241 U1
-U 1 1 546B4692
-P 3800 3200
-F 0 "U1" H 3800 3350 60  0000 L CNN
-F 1 "MCP6241" H 3800 3050 60  0000 L CNN
-F 2 "~" H 3800 3200 60  0000 C CNN
-F 3 "~" H 3800 3200 60  0000 C CNN
-	1    3800 3200
+L MCP6242 U2
+U 2 1 54906D15
+P 3900 3200
+F 0 "U2" H 4000 3400 60  0000 L CNN
+F 1 "MCP6242" H 3950 3000 60  0000 L CNN
+F 2 "~" H 4000 3200 60  0000 C CNN
+F 3 "~" H 4000 3200 60  0000 C CNN
+	2    3900 3200
 	-1   0    0    -1
 $EndComp
-Text HLabel 5700 3100 2    60   Input ~ 0
-pH_ProbeIN
 $EndSCHEMATC
