File: Kicad/pH.sch (KiCad schematic (older format))
At the start: 1 part, among them U2 MCP6242

Commit message: check in before modifying Layout with updated design
Parts:
- removed U2: MCP6242, ~, symbol MCP6242
- added U?: MCP6241, ~, symbol MCP6241
Connections:
- net labels added: Vclean
- wire segments 8 -> 12
Changed lines of the file:
@@
 Sheet 4 11
 Title ""
-Date "29 jan 2015"
+Date "31 jan 2015"
 Rev ""
 Comp ""
@@
 VGND
 $Comp
-L MCP6242 U2
-U 2 1 54906D15
-P 3900 3200
-F 0 "U2" H 4000 3400 60  0000 L CNN
-F 1 "MCP6242" H 3950 3000 60  0000 L CNN
-F 2 "~" H 4000 3200 60  0000 C CNN
-F 3 "~" H 4000 3200 60  0000 C CNN
-	2    3900 3200
-	-1   0    0    -1
+L MCP6241 U?
+U 1 1 54CCCA62
+P 3800 3200
+F 0 "U?" H 3800 3350 60  0000 L CNN
+F 1 "MCP6241" H 3800 3050 60  0000 L CNN
+F 2 "~" H 3800 3200 60  0000 C CNN
+F 3 "~" H 3800 3200 60  0000 C CNN
+	1    3800 3200
+	-1   0    0    1
 $EndComp
+Wire Wire Line
+	3900 3500 3900 3700
+Wire Wire Line
+	3900 3700 3800 3700
+Text GLabel 1750 2550 0    60   Input ~ 0
+Vclean
+Wire Wire Line
+	1750 2550 3900 2550
+Wire Wire Line
+	3900 2550 3900 2900
 $EndSCHEMATC

Commit message: first pass at new layout
Parts:
- gave numbers to parts that had none: 1
Connections:
- net labels added: GND
Changed lines of the file:
@@
 Sheet 4 11
 Title ""
-Date "31 jan 2015"
+Date "2 feb 2015"
 Rev ""
 Comp ""
@@
 VGND
 $Comp
-L MCP6241 U?
+L MCP6241 U1
 U 1 1 54CCCA62
 P 3800 3200
-F 0 "U?" H 3800 3350 60  0000 L CNN
+F 0 "U1" H 3800 3350 60  0000 L CNN
 F 1 "MCP6241" H 3800 3050 60  0000 L CNN
 F 2 "~" H 3800 3200 60  0000 C CNN
@@
 Wire Wire Line
 	3900 2550 3900 2900
+Text GLabel 3800 3700 0    60   Input ~ 0
+GND
 $EndSCHEMATC
