File: Kicad/ECGain.sch (KiCad schematic (older format))
At the start: 3 parts, among them U5 MCP6244

Commit message: iPhone app and changes to hw design (not sure I like)
Connections:
- net labels added: EC_VIN, EC_VOUT
- net labels removed: EC_DCv, EC_Vin+
Changed lines of the file:
@@
 $Descr A4 11693 8268
 encoding utf-8
-Sheet 7 11
+Sheet 7 9
 Title ""
-Date "9 feb 2015"
+Date "17 mar 2015"
 Rev ""
 Comp ""
@@
 GND
 Text HLabel 3450 3000 0    60   Input ~ 0
-EC_Vin+
+EC_VIN
 Wire Wire Line
 	3450 3000 5650 3000
 Text HLabel 7850 3100 2    60   Output ~ 0
-EC_DCv
+EC_VOUT
 $EndSCHEMATC
