File: Kicad/ECGain.sch (KiCad schematic (older format))
At the start: 3 parts

Commit message: layout for Alpha 2
Parts:
- gave numbers to parts that had none: 3
Changed lines of the file:
@@
 Sheet 7 11
 Title ""
-Date "29 jan 2015"
+Date "8 feb 2015"
 Rev ""
 Comp ""
@@
 	5100 5300 4950 5300
 $Comp
-L MCP6244 U?
+L MCP6244 U5
 U 1 1 54C7A596
 P 5900 3100
-F 0 "U?" H 6000 3300 60  0000 L CNN
+F 0 "U5" H 6000 3300 60  0000 L CNN
 F 1 "MCP6244" H 5950 2900 60  0000 L CNN
 F 2 "~" H 6000 3100 60  0000 C CNN
@@
 Connection ~ 5450 4050
 $Comp
-L R R?
+L R R17
 U 1 1 54C7A5A6
 P 6100 4050
-F 0 "R?" V 6180 4050 40  0000 C CNN
+F 0 "R17" V 6180 4050 40  0000 C CNN
 F 1 "1K .5%" V 6107 4051 40  0000 C CNN
 F 2 "~" V 6030 4050 30  0000 C CNN
@@
 $EndComp
 $Comp
-L C C?
+L C C6
 U 1 1 54C7A5AC
 P 6150 2550
-F 0 "C?" H 6150 2650 40  0000 L CNN
+F 0 "C6" H 6150 2650 40  0000 L CNN
 F 1 ".1u" H 6156 2465 40  0000 L CNN
 F 2 "~" H 6188 2400 30  0000 C CNN

Commit message: Beta 2 sent to OSHPark
Connections:
- net labels added: EC_Vin, EC_Vout
- net labels removed: EC_DCv, EC_Vin+
Changed lines of the file:
@@
 $Descr A4 11693 8268
 encoding utf-8
-Sheet 7 11
+Sheet 7 10
 Title ""
-Date "9 feb 2015"
+Date "26 mar 2015"
 Rev ""
 Comp ""
@@
 GND
 Text HLabel 3450 3000 0    60   Input ~ 0
-EC_Vin+
+EC_Vin
 Wire Wire Line
 	3450 3000 5650 3000
 Text HLabel 7850 3100 2    60   Output ~ 0
-EC_DCv
+EC_Vout
 $EndSCHEMATC
