File: Kicad/Rectify.sch (KiCad schematic (older format))
At the start: 5 parts

Commit message: layout for Alpha 2
Parts:
- gave numbers to parts that had none: 4
Connections:
- net RVin-: now also U5.9 (-); no longer U5.6 (-)
- net R_Vout: now also U5.8; no longer U5.7
- net Signal: now also U5.10 (+); no longer U5.5 (+)
- net R_Drain renamed FET_pin
Changed lines of the file:
@@
 Sheet 8 11
 Title ""
-Date "29 jan 2015"
+Date "8 feb 2015"
 Rev ""
 Comp ""
@@
 $EndDescr
 $Comp
-L DIODE D?
+L DIODE D7
 U 1 1 54C7CC9B
 P 4850 3300
-F 0 "D?" H 4850 3400 40  0000 C CNN
+F 0 "D7" H 4850 3400 40  0000 C CNN
 F 1 "DIODE" H 4850 3200 40  0000 C CNN
 F 2 "~" H 4850 3300 60  0000 C CNN
@@
 $EndComp
 $Comp
-L C C?
+L C C7
 U 1 1 54C7CCA1
 P 5700 3550
-F 0 "C?" H 5700 3650 40  0000 L CNN
+F 0 "C7" H 5700 3650 40  0000 L CNN
 F 1 ".1u" H 5706 3465 40  0000 L CNN
 F 2 "~" H 5738 3400 30  0000 C CNN
@@
 	2400 3200 3800 3200
 $Comp
-L MCP6244 U?
-U 2 1 54C7CCAB
+L MCP6244 U5
+U 3 1 54C7CCAB
 P 4050 3300
-F 0 "U?" H 4150 3500 60  0000 L CNN
+F 0 "U5" H 4150 3500 60  0000 L CNN
 F 1 "MCP6244" H 4100 3100 60  0000 L CNN
 F 2 "~" H 4150 3300 60  0000 C CNN
 F 3 "~" H 4150 3300 60  0000 C CNN
-	2    4050 3300
+	3    4050 3300
 	1    0    0    -1
 $EndComp
@@
 VGND
 $Comp
-L MCP6244 U?
+L MCP6244 U5
 U 4 1 54C7CCD8
 P 7000 3400
-F 0 "U?" H 7100 3600 60  0000 L CNN
+F 0 "U5" H 7100 3600 60  0000 L CNN
 F 1 "MCP6244" H 7050 3200 60  0000 L CNN
 F 2 "~" H 7100 3400 60  0000 C CNN
@@
 Connection ~ 5700 3300
 $Comp
-L MOSFET_N Q?
+L MOSFET_N Q4
 U 1 1 54C8E8C1
 P 6250 3700
-F 0 "Q?" H 6260 3870 60  0000 R CNN
+F 0 "Q4" H 6260 3870 60  0000 R CNN
 F 1 "MOSFET_N" H 6260 3550 60  0000 R CNN
 F 2 "~" H 6250 3700 60  0000 C CNN
@@
 	6050 4550 2450 4550
 Text HLabel 2450 4550 0    100  Input ~ 0
-R_Drain
+FET_pin
 $EndSCHEMATC
