File: Kicad/Rectify.sch (KiCad schematic (older format))
At the start: 4 parts, among them Q4 MOSFET_N, U5 MCP6244

Commit message: minor changes - all works
Parts:
- removed Q4: MOSFET_N, ~, symbol MOSFET_N
- added Q4: LB_MOSFET_N, ~, symbol LB_MOSFET_N
Connections:
- net FET_pin: now also Q4.G
- net RVin-: now also Q4.D
- net VGND: now also Q4.S
Changed lines of the file:
@@
 Sheet 8 10
 Title ""
-Date "26 mar 2015"
+Date "13 apr 2015"
 Rev ""
 Comp ""
@@
 Connection ~ 5350 3300
 Connection ~ 5700 3300
-$Comp
-L MOSFET_N Q4
-U 1 1 54C8E8C1
-P 6250 3700
-F 0 "Q4" H 6260 3870 60  0000 R CNN
-F 1 "MOSFET_N" H 6260 3550 60  0000 R CNN
-F 2 "~" H 6250 3700 60  0000 C CNN
-F 3 "~" H 6250 3700 60  0000 C CNN
-	1    6250 3700
-	1    0    0    -1
-$EndComp
 Wire Wire Line
 	6350 3500 6350 3300
@@
 Text HLabel 2450 4550 0    100  Input ~ 0
 FET_pin
+$Comp
+L LB_MOSFET_N Q4
+U 1 1 552BD149
+P 6250 3700
+F 0 "Q4" H 6260 3870 60  0000 R CNN
+F 1 "LB_MOSFET_N" H 6260 3550 60  0000 R CNN
+F 2 "~" H 6250 3700 60  0000 C CNN
+F 3 "~" H 6250 3700 60  0000 C CNN
+	1    6250 3700
+	1    0    0    -1
+$EndComp
 $EndSCHEMATC
