File: Kicad/_autosave-LadyBugShield.kicad_pcb (KiCad board)
At the start: 2 copper layers, 88.1 x 55.3 mm, 55 parts, among them P1 CONN_6, P2 CONN_2, P5 CONN_2, Q1 TIP122, Q2 TIP122, Q3 TIP122, Q4 MOSFET_N, U1 74LVC1G53, U2 MCP6242, U4 ADS1015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

Commit message: Beta 2 sent to OSHPark
Parts:
- moved ? 13.6 mm to (190.2, 75.0)
- moved ? 4.99 mm to (180.5, 99.5)
Other:
- board text added: "Beta 2"
- board text removed: "Alpha V2"
