File: Kicad/AC.sch (KiCad schematic (older format))
At the start: 12 parts

Commit message: layout for Alpha 2
Parts:
- C2, C3, C5: renamed from C?; value 100n -> .1u
- gave numbers to parts that had none: 9
Connections:
- net W_Vin+: now also U5.5 (+); no longer U5.10 (+)
- net W_Vin-: now also U5.6 (-); no longer U5.9 (-)
- net W_Vout: now also U5.7; no longer U5.8
Changed lines of the file:
@@
 Sheet 6 11
 Title ""
-Date "29 jan 2015"
+Date "8 feb 2015"
 Rev ""
 Comp ""
@@
 $EndDescr
 $Comp
-L R R?
+L R R3
 U 1 1 54C79AB8
 P 4650 3750
-F 0 "R?" V 4730 3750 40  0000 C CNN
+F 0 "R3" V 4730 3750 40  0000 C CNN
 F 1 "1K" V 4657 3751 40  0000 C CNN
 F 2 "~" V 4580 3750 30  0000 C CNN
@@
 $EndComp
 $Comp
-L R R?
+L R R4
 U 1 1 54C79ABE
 P 4800 4950
-F 0 "R?" V 4880 4950 40  0000 C CNN
+F 0 "R4" V 4880 4950 40  0000 C CNN
 F 1 "10K" V 4807 4951 40  0000 C CNN
 F 2 "~" V 4730 4950 30  0000 C CNN
@@
 $EndComp
 $Comp
-L C C?
+L C C2
 U 1 1 54C79AC4
 P 4700 3150
-F 0 "C?" H 4700 3250 40  0000 L CNN
-F 1 "100n" H 4706 3065 40  0000 L CNN
+F 0 "C2" H 4700 3250 40  0000 L CNN
+F 1 ".1u" H 4706 3065 40  0000 L CNN
 F 2 "~" H 4738 3000 30  0000 C CNN
 F 3 "~" H 4700 3150 60  0000 C CNN
@@
 $EndComp
 $Comp
-L C C?
+L C C3
 U 1 1 54C79ACA
 P 6100 5750
-F 0 "C?" H 6100 5850 40  0000 L CNN
-F 1 "100n" H 6106 5665 40  0000 L CNN
+F 0 "C3" H 6100 5850 40  0000 L CNN
+F 1 ".1u" H 6106 5665 40  0000 L CNN
 F 2 "~" H 6138 5600 30  0000 C CNN
 F 3 "~" H 6100 5750 60  0000 C CNN
@@
 $EndComp
 $Comp
-L DIODE D?
+L DIODE D4
 U 1 1 54C79AD0
 P 5500 5600
-F 0 "D?" H 5500 5700 40  0000 C CNN
+F 0 "D4" H 5500 5700 40  0000 C CNN
 F 1 "DIODE" H 5500 5500 40  0000 C CNN
 F 2 "~" H 5500 5600 60  0000 C CNN
@@
 $EndComp
 $Comp
-L DIODE D?
+L DIODE D6
 U 1 1 54C79AD6
 P 5500 5900
-F 0 "D?" H 5500 6000 40  0000 C CNN
+F 0 "D6" H 5500 6000 40  0000 C CNN
 F 1 "DIODE" H 5500 5800 40  0000 C CNN
 F 2 "~" H 5500 5900 60  0000 C CNN
@@
 $EndComp
 $Comp
-L C C?
+L C C5
 U 1 1 54C79ADC
 P 6450 3450
-F 0 "C?" H 6450 3550 40  0000 L CNN
-F 1 "100n" H 6456 3365 40  0000 L CNN
+F 0 "C5" H 6450 3550 40  0000 L CNN
+F 1 ".1u" H 6456 3365 40  0000 L CNN
 F 2 "~" H 6488 3300 30  0000 C CNN
 F 3 "~" H 6450 3450 60  0000 C CNN
@@
 $EndComp
 $Comp
-L R R?
+L R R13
 U 1 1 54C79AE2
 P 6050 3150
-F 0 "R?" V 6130 3150 40  0000 C CNN
+F 0 "R13" V 6130 3150 40  0000 C CNN
 F 1 "1K" V 6057 3151 40  0000 C CNN
 F 2 "~" V 5980 3150 30  0000 C CNN
@@
 $EndComp
 $Comp
-L R R?
+L R R14
 U 1 1 54C79AE8
 P 6900 3850
-F 0 "R?" V 7000 3850 40  0000 C CNN
+F 0 "R14" V 7000 3850 40  0000 C CNN
 F 1 "10K" V 6907 3851 40  0000 C CNN
 F 2 "~" V 6830 3850 30  0000 C CNN
@@
 	7150 3850 8400 3850
 $Comp
-L MCP6244 U?
-U 3 1 54C79AFF
+L MCP6244 U5
+U 2 1 54C79AFF
 P 5650 3850
-F 0 "U?" H 5750 4050 60  0000 L CNN
+F 0 "U5" H 5750 4050 60  0000 L CNN
 F 1 "MCP6244" H 5700 3650 60  0000 L CNN
 F 2 "~" H 5750 3850 60  0000 C CNN
 F 3 "~" H 5750 3850 60  0000 C CNN
-	3    5650 3850
+	2    5650 3850
 	1    0    0    -1
 $EndComp
@@
 	7450 2900 7450 2700
 $Comp
-L R R?
+L R R12
 U 1 1 54C79B28
 P 5800 4850
-F 0 "R?" V 5880 4850 40  0000 C CNN
+F 0 "R12" V 5880 4850 40  0000 C CNN
 F 1 "22K" V 5807 4851 40  0000 C CNN
 F 2 "~" V 5730 4850 30  0000 C CNN
@@
 $EndComp
 $Comp
-L R R?
+L R R16
 U 1 1 54C79B2E
 P 7450 3150
-F 0 "R?" V 7530 3150 40  0000 C CNN
+F 0 "R16" V 7530 3150 40  0000 C CNN
 F 1 "10K" V 7457 3151 40  0000 C CNN
 F 2 "~" V 7380 3150 30  0000 C CNN

Commit message: Beta 2 sent to OSHPark
Connections:
- net EC_Vin+ renamed EC_Vin
Changed lines of the file:
@@
 $Descr A4 11693 8268
 encoding utf-8
-Sheet 6 11
+Sheet 6 10
 Title ""
-Date "9 feb 2015"
+Date "26 mar 2015"
 Rev ""
 Comp ""
@@
 VGND
 Text HLabel 8400 3850 2    60   Output ~ 0
-EC_Vin+
+EC_Vin
 $EndSCHEMATC
