File: Kicad/LadyBugShield.kicad_pcb (KiCad board)
At the start: 2 copper layers, 81.3 x 55.3 mm, 52 parts, among them P1 CONN_6, P2 CONN_2, P3 BNC, P4 BNC, Q1 TIP122, Q2 TIP122, Q3 TIP122, Q4 MOSFET_N, U1 74LVC1G53, U2 MCP6242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

Commit message: Beta 2 sent to OSHPark
Parts:
- removed C11: 1u, SM0805
- removed C12: 10u, SM0805
- removed C13: .1u, SM0805
- removed R15: 10K 1%, SM0805
- removed U3: MC78L05, LB_SOT89_3
- added D8: LED, SM1206, F.Cu at (173.9, 106.5)
- added P5: CONN_2, LB_CONN_2, F.Cu at (172.1, 113.1)
- added TP1: Vin, LB_TestPoint, F.Cu at (217.3, 102.2)
- added TP2: pH_AIN, LB_TestPoint, F.Cu at (226.6, 98.9)
- added TP3: EC_AIN, LB_TestPoint, F.Cu at (223.2, 97.4)
- added TP4: Vout, LB_TestPoint, F.Cu at (211.6, 107.6)
- added VGND_TP1: CONN_1, LB_TestPoint, F.Cu at (226.3, 81.7)
- added VP1: S, LB_TestPoint, F.Cu at (198.2, 102.0)
- ARD1: value ARDUINOPINS -> (none)
- R2: value 10K -> 1K
- moved P2 76.4 mm to (162.2, 113.2), turned to 180 degrees
- moved R2 35.4 mm to (171.4, 103.2), turned to 0 degrees
- moved D3 30.5 mm to (194.7, 106.4), turned to 180 degrees
- moved R5 21.0 mm to (189.2, 106.5), turned to 0 degrees
- moved PH 8.01 mm to (231.4, 82.0)
- moved R13 7.28 mm to (203.8, 90.4)
- moved EC 6.80 mm to (231.7, 100.5)
- moved R4 6.78 mm to (203.5, 82.2), turned to 90 degrees
- moved R9 6.52 mm to (201.6, 75.7)
- moved C8 6.48 mm to (219.4, 99.6)
- moved U4 5.77 mm to (223.3, 104.4)
- moved R7 5.77 mm to (226.6, 108.6)
- moved C7 5.47 mm to (189.7, 95.9)
- moved D7 5.47 mm to (190.9, 90.4)
- moved Q4 5.47 mm to (190.5, 99.4)
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- renumbered P4 to EC, P3 to PH
Connections:
- net /Arduino/Pump1 renamed /Arduino/pump1_pin
- net /Arduino/Pump2 renamed /Arduino/pump2_pin
- net /Arduino/Pump3 renamed /Arduino/pump3_pin
- net /EC/AC/EC_Vin+ renamed /EC/AC/EC_Vin
- net /EC/ECGain/EC_DCv renamed /EC/ECGain/EC_Vout
- net /Pumps/SW_Pump1 renamed /Pumps/pump1
- net /Pumps/SW_Pump2 renamed /Pumps/pump2
- net /Pumps/SW_Pump3 renamed /Pumps/pump3
- ARD1 pad 1: (no net) -> Vclean
- ARD1 pad 4: Vin -> /Arduino/12V
- ARD1 pad 7: /Arduino/MUX_enable_pin -> (no net)
- C1 pad 1: VClean -> Vclean
- C4 pad 1: VClean -> Vclean
- C6 pad 1: VClean -> Vclean
- C8 pad 1: VClean -> Vclean
- C9 pad 1: VClean -> Vclean
- D1 pad 2: VClean -> /Arduino/12V
- D2 pad 2: VClean -> /Arduino/12V
- D3 pad 1: VClean -> Vclean
- D5 pad 2: VClean -> /Arduino/12V
- P1 pad 1: VClean -> /Arduino/12V
- P1 pad 3: VClean -> /Arduino/12V
- P1 pad 5: VClean -> /Arduino/12V
- P2 pad 1: /DigitalAccess/Therm_AIN -> /Arduino/12Va
- P2 pad 2: VClean -> GND
- R2 pad 1: /Arduino/MUX_enable_pin -> GND
- R2 pad 2: VClean -> N-0000019
- R6 pad 1: VClean -> Vclean
- R7 pad 1: VClean -> Vclean
- R8 pad 1: VClean -> Vclean
- U1 pad 2: /Arduino/MUX_enable_pin -> GND
- U1 pad 8: VClean -> Vclean
- U2 pad 8: VClean -> Vclean
- U4 pad 6: /DigitalAccess/Therm_AIN -> (no net)
- U4 pad 8: VClean -> Vclean
- U5 pad 4: VClean -> Vclean
Routing:
- net VClean: track 320.1 -> 0.00 mm, vias 2 -> 0
- net Vclean: track 0.00 -> 207.6 mm
- net /Arduino/12V: track 0.00 -> 103.1 mm
- net Vin: track 33.0 -> 0.00 mm
- net /DigitalAccess/Therm_AIN: track 30.7 -> 0.00 mm, vias 2 -> 0
- net VGND: track 149.8 -> 125.8 mm, vias 1 -> 0
- net /DigitalAccess/EC_AIN: track 21.9 -> 40.6 mm, vias 2 -> 1
- net /DigitalAccess/pH_AIN: track 83.6 -> 66.2 mm, vias 2 -> 1
- net /Arduino/MUX_enable_pin: track 16.3 -> 0.00 mm
- net /EC/EC_ProbeIN: track 21.4 -> 37.2 mm, vias 0 -> 2
- net /Power/VGND_V+: track 10.5 -> 23.7 mm
- net GND: track 46.7 -> 34.2 mm, vias 17 -> 15
- net /EC/AC/EC_Vin: track 25.1 -> 36.1 mm
- net /pH/pH_ProbeIN: track 10.9 -> 21.5 mm
- net /EC/ECGain/EC_Vout: track 18.3 -> 27.6 mm
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Other:
- board size 81.3 x 55.3 mm -> 88.1 x 55.3 mm

Commit message: Initial Commit
Parts:
- moved ? 13.6 mm to (190.2, 75.0)
- moved ? 4.99 mm to (180.5, 99.5)
Other:
- board text added: "Beta 2"
- board text removed: "Alpha V2"

Commit message: minor changes - all works
Parts:
- removed D3: LED, SM1206
- removed P2, P5: CONN_2, LB_CONN_2
- removed R5: 1K, SM0805
- ARD1: value (none) -> ARDUINOPINS
- Q4: value MOSFET_N -> LB_MOSFET_N
- moved D8 3.15 mm to (170.8, 107.0)
- moved R2 1.41 mm to (170.0, 103.0), turned to 180 degrees
- moved Q4 0.16 mm to (190.5, 99.3)
- renumbered PH to P3, EC to P4, VP1 to TP_S, VGND_TP1 to TP_VGND, TP1 to TP_VIN, TP4 to TP_VOUT
Routing:
- net /Arduino/12Va: track 6.66 -> 0.00 mm
- net /Arduino/12V: track 103.1 -> 99.2 mm
- net N-0000047: track 3.00 -> 0.00 mm
- net GND: track 34.2 -> 31.7 mm, vias 15 -> 14
- net N-0000020: track 3.37 -> 4.05 mm
Other:
- board text added: "EC"
- board text added: "pH"
