File: Kicad/LadyBugShield.sch (KiCad schematic (older format))
At the start: 4 parts, among them P1 CONN_6, P2 CONN_2, P3 BNC, P4 BNC

Commit message: Beta 2 sent to OSHPark
Parts:
- removed P2: CONN_2, symbol CONN_2
- added TP2: pH_AIN, symbol CONN_1
- added TP3: EC_AIN, symbol CONN_1
Connections:
- net Pumps/V+_Pump2 is gone; now on net Arduino/12V: P1.3
- net Pumps/V+_Pump3 is gone; now on net Arduino/12V: P1.5
- net DigitalAccess/EC_AIN: now also TP3.1
- net DigitalAccess/pH_AIN: now also TP2.1
- net Pumps/SW_Pump1 renamed Pumps/pump1
- net Pumps/SW_Pump2 renamed Pumps/pump2
- net Pumps/SW_Pump3 renamed Pumps/pump3
- net Pumps/V+_Pump1 renamed Arduino/12V
Other:
- moved on the sheet: P1, P4
Changed lines of the file:
@@
 $Descr A4 11693 8268
 encoding utf-8
-Sheet 1 11
+Sheet 1 10
 Title ""
-Date "9 feb 2015"
+Date "26 mar 2015"
 Rev ""
 Comp ""
@@
 F2 "SDA" B R 3300 2400 60
 F3 "SCL" O R 3300 2200 60
-F4 "Pump2" O R 3300 5650 60
-F5 "Pump1" O R 3300 5450 60
-F6 "Pump3" O R 3300 5850 60
-F7 "MUX_out_pin" O R 3300 4250 60
-F8 "FET_pin" O R 3300 4450 60
-F9 "MUX_enable_pin" O R 3300 4050 60
+F4 "pump2_pin" O R 3300 5650 60
+F5 "pump1_pin" O R 3300 5450 60
+F6 "pump3_pin" O R 3300 5850 60
+F7 "MUX_out_pin" O R 3300 3950 60
+F8 "FET_pin" O R 3300 4150 60
+F9 "12V" O R 3300 5250 60
 $EndSheet
 $Sheet
@@
 F4 "pH_AIN" I R 5950 2050 60
 F5 "EC_AIN" I R 5950 3550 60
-F6 "Therm_AIN" I R 5950 2700 60
 $EndSheet
 $Sheet
@@
 $EndSheet
 $Sheet
-S 6750 3600 2600 1000
+S 6950 3300 2600 1000
 U 547DE5B0
 F0 "EC" 50
 F1 "EC.sch" 50
-F2 "EC_ProbeIN" I R 9350 3950 60
-F3 "EC_AIN" O L 6750 3850 60
-F4 "MUX_out_pin" I L 6750 4250 60
-F5 "FET_pin" I L 6750 4450 60
-F6 "MUX_enable_pin" I L 6750 4050 60
+F2 "EC_ProbeIN" I R 9550 3650 60
+F3 "EC_AIN" O L 6950 3550 60
+F4 "MUX_out_pin" I L 6950 3950 60
+F5 "FET_pin" I L 6950 4150 60
 $EndSheet
 $Sheet
@@
 Wire Wire Line
 	9300 1250 10550 1250
-Wire Wire Line
-	9400 2700 10200 2700
 Wire Wire Line
 	6750 1250 6600 1250
@@
 	3300 2400 4050 2400
 Connection ~ 6350 6850
-$Sheet
-S 6750 2400 2650 950
-U 547DE6A0
-F0 "Temperature" 50
-F1 "Temperature.sch" 50
-F2 "Therm_IN" I R 9400 2700 60
-F3 "Therm_AIN" O L 6750 2700 60
-$EndSheet
 Text GLabel 10700 1700 0    60   Input ~ 0
 VGND
-Text GLabel 10700 4300 0    60   Input ~ 0
+Text GLabel 10900 4000 0    60   Input ~ 0
 VGND
-Text GLabel 9950 2900 0    60   Input ~ 0
-Vclean
 $Comp
 L BNC P3
@@
 L BNC P4
 U 1 1 54903E31
-P 10700 3950
-F 0 "P4" H 10710 4070 60  0000 C CNN
-F 1 "BNC" V 10810 3890 40  0000 C CNN
-F 2 "~" H 10700 3950 60  0000 C CNN
-F 3 "~" H 10700 3950 60  0000 C CNN
-	1    10700 3950
-	1    0    0    -1
-$EndComp
-$Comp
-L CONN_2 P2
-U 1 1 54903E39
-P 10550 2800
-F 0 "P2" V 10500 2800 40  0000 C CNN
-F 1 "CONN_2" V 10600 2800 40  0000 C CNN
-F 2 "" H 10550 2800 60  0000 C CNN
-F 3 "" H 10550 2800 60  0000 C CNN
-	1    10550 2800
+P 10900 3650
+F 0 "P4" H 10910 3770 60  0000 C CNN
+F 1 "BNC" V 11010 3590 40  0000 C CNN
+F 2 "~" H 10900 3650 60  0000 C CNN
+F 3 "~" H 10900 3650 60  0000 C CNN
+	1    10900 3650
 	1    0    0    -1
 $EndComp
@@
 L CONN_6 P1
 U 1 1 54903E48
-P 6900 5550
-F 0 "P1" V 6850 5550 60  0000 C CNN
-F 1 "CONN_6" V 6950 5550 60  0000 C CNN
-F 2 "" H 6900 5550 60  0000 C CNN
-F 3 "" H 6900 5550 60  0000 C CNN
-	1    6900 5550
+P 7750 5850
+F 0 "P1" V 7700 5850 60  0000 C CNN
+F 1 "CONN_6" V 7800 5850 60  0000 C CNN
+F 2 "" H 7750 5850 60  0000 C CNN
+F 3 "" H 7750 5850 60  0000 C CNN
+	1    7750 5850
 	1    0    0    -1
 $EndComp
@@
 	10700 1450 10700 1700
 Wire Wire Line
-	10550 3950 9350 3950
+	10750 3650 9550 3650
 Wire Wire Line
-	10700 4150 10700 4300
+	10900 3850 10900 4000
 Wire Wire Line
 	3300 5450 4400 5450
@@
 Wire Wire Line
 	3300 5850 4400 5850
+Wire Wire Line
+	6050 5700 7400 5700
+Wire Wire Line
+	6650 5800 7400 5800
+Wire Wire Line
+	6050 5900 7400 5900
+Wire Wire Line
+	6650 6000 7400 6000
+Wire Wire Line
+	6050 6100 7400 6100
+Wire Wire Line
+	3300 3950 6950 3950
+Wire Wire Line
+	3300 5250 4400 5250
 $Sheet
 S 4400 5100 1650 1300
@@
 F0 "Pumps" 50
 F1 "Pumps.sch" 50
-F2 "Pump1" I L 4400 5450 60
-F3 "V+_Pump1" I R 6050 5300 60
-F4 "SW_Pump1" I R 6050 5400 60
-F5 "Pump2" I L 4400 5650 60
-F6 "SW_Pump2" I R 6050 5600 60
-F7 "V+_Pump2" I R 6050 5500 60
-F8 "Pump3" I L 4400 5850 60
-F9 "SW_Pump3" I R 6050 5800 60
-F10 "V+_Pump3" I R 6050 5700 60
+F2 "pump2_pin" I L 4400 5650 60
+F3 "pump3_pin" I L 4400 5850 60
+F4 "pump1_pin" I L 4400 5450 60
+F5 "12V" I L 4400 5250 60
+F6 "pump1" O R 6050 5700 60
+F7 "pump2" O R 6050 5900 60
+F8 "pump3" O R 6050 6100 60
 $EndSheet
 Wire Wire Line
-	9950 2900 10200 2900
+	6650 4850 6650 6000
 Wire Wire Line
-	6550 5300 6050 5300
+	7400 5600 6650 5600
+Connection ~ 6650 5600
+Connection ~ 6650 5800
 Wire Wire Line
-	6050 5400 6550 5400
+	3850 5250 3850 4850
 Wire Wire Line
-	6050 5500 6550 5500
+	3850 4850 6650 4850
+Connection ~ 3850 5250
+$Comp
+L CONN_1 TP2
+U 1 1 5513E844
+P 6450 2400
+F 0 "TP2" H 6530 2400 40  0001 L CNN
+F 1 "pH_AIN" H 6450 2455 30  0000 C CNN
+F 2 "" H 6450 2400 60  0000 C CNN
+F 3 "" H 6450 2400 60  0000 C CNN
+	1    6450 2400
+	1    0    0    -1
+$EndComp
+$Comp
+L CONN_1 TP3
+U 1 1 5513E851
+P 6550 3100
+F 0 "TP3" H 6630 3100 40  0001 L CNN
+F 1 "EC_AIN" H 6550 3155 30  0000 C CNN
+F 2 "" H 6550 3100 60  0000 C CNN
+F 3 "" H 6550 3100 60  0000 C CNN
+	1    6550 3100
+	1    0    0    -1
+$EndComp
 Wire Wire Line
-	6050 5600 6550 5600
+	6300 2400 6300 2050
+Connection ~ 6300 2050
 Wire Wire Line
-	6050 5700 6550 5700
+	5950 3550 6950 3550
 Wire Wire Line
-	6050 5800 6550 5800
+	3300 4150 6950 4150
 Wire Wire Line
-	5950 2700 6750 2700
-Wire Wire Line
-	6750 3850 6300 3850
-Wire Wire Line
-	6300 3850 6300 3550
-Wire Wire Line
-	6300 3550 5950 3550
-Wire Wire Line
-	3300 4050 6750 4050
-Wire Wire Line
-	3300 4250 6750 4250
-Wire Wire Line
-	3300 4450 6750 4450
+	6400 3100 6400 3550
+Connection ~ 6400 3550
 $EndSCHEMATC
