File: LBS-TEST1/LBS-TEST1.sch (KiCad schematic (older format))
At the start: 8 parts, among them P1 CONN_1, P10 CONN_1, P2 CONN_1, P3 CONN_1, P4 CONN_1, P7 CONN_1, P8 CONN_1, P9 CONN_1

Commit message: added switch circuits for rectifier for discussion
Other:
- note added: "demultiplex"
Changed lines of the file:
@@
 Sheet 1 5
 Title ""
-Date "15 jan 2015"
+Date "26 jan 2015"
 Rev ""
 Comp ""
@@
 D9 E2 BF C4 18 F7 0C 4B 5E B4 8D 6F 67 A1 70 71 C5 12 A3 BD DD C9 B3 93 77 93 9B 2B F6 BC 6A 4C
 31 A6 9D A4 5C 5A 6D B5 D5 56 5B 6D B5 D5 02 ED 0F 8F D8 15 DB 22 89 0B B4 00 00 00 00 49 45 4E
-44 AE 42 60 82 27 $EndBitmap
+44 AE 42 60 82 29 $EndBitmap
 EndData
 $EndBitmap
@@
 12 D7 1E 39 D3 97 8B E9 CC 09 7E A4 21 84 7B DE 75 BE 6C 10 1D B1 C0 C8 E6 44 20 98 58 88 D3 4B
 BF A4 FE AC E7 27 87 F5 F3 E7 B2 6E 04 7A D3 5E FF 1F 0B 1A 44 E2 12 6D EC E1 00 00 00 00 49 45
-4E 44 AE 42 60 82 74 $EndBitmap
+4E 44 AE 42 60 82 75 $EndBitmap
 EndData
 $EndBitmap
@@
 68 8C 04 22 37 29 8A 92 CF E7 4D D3 14 0F B2 A5 52 A9 64 32 99 CF E7 BD 2E 17 51 47 38 08 95 88
 88 2C AC 25 10 11 91 85 91 40 44 44 16 46 02 11 11 59 18 09 44 44 64 61 24 10 11 91 85 91 40 44
-44 96 FF 0F 99 70 A1 25 65 0E B8 12 00 00 00 00 49 45 4E 44 AE 42 60 82 03 $EndBitmap
+44 96 FF 0F 99 70 A1 25 65 0E B8 12 00 00 00 00 49 45 4E 44 AE 42 60 82 92 $EndBitmap
 EndData
 $EndBitmap
@@
 Wire Notes Line
 	3350 1700 5750 1700
+Wire Notes Line
+	3200 2900 3200 5000
+Wire Notes Line
+	5600 2800 5600 4700
+Wire Notes Line
+	5600 4700 6600 4700
+Wire Notes Line
+	6600 4700 6600 4650
+Wire Notes Line
+	7350 4700 7350 4100
+Wire Notes Line
+	7350 4100 5750 4100
+Wire Notes Line
+	5750 4100 5750 2850
+Wire Notes Line
+	7000 4500 6600 4500
+Wire Notes Line
+	6600 4500 6600 5000
+Wire Notes Line
+	7000 4500 7000 5250
+Wire Notes Line
+	7000 5250 6600 5250
+Wire Notes Line
+	6600 5250 6600 4950
+Wire Notes Line
+	7000 4700 7350 4700
+Wire Notes Line
+	6600 5000 3200 5000
+Text Notes 7350 5050 0    100  ~ 0
+demultiplex
 $EndSCHEMATC
